File: PCB and Schem/HyperPlex.kicad_sch (KiCad schematic)
At the start: 23 parts, among them Q1 2N3904, Q2 2N3904, U1 CH32V203CxTx, U2 GD25QxxxEY, U3 XC6206PxxxMR, U4 TP4056-42-ESOP8, U5 TPS63900

Commit message: Added USB Jack, Power switch, and Reset button to schematic
Parts:
- added J1: USB_C_Receptacle_USB2.0_16P, symbol Connector:USB_C_Receptacle_USB2.0_16P
- added Q3: 2N3904, Package_TO_SOT_SMD:SOT-23, symbol Transistor_BJT:2N3904
- added R12, R13: 5.1k, Resistor_SMD:R_0603_1608Metric, symbol Device:R
- added R15: 500, Resistor_SMD:R_0603_1608Metric, symbol Device:R
- added SW1: SW_Push, symbol Switch:SW_Push
- added SW2: SW_SPDT, symbol Switch:SW_SPDT
- C1, C2, L1, R10, R11, R7, R8, R9, U5: now not fitted; now left out of the parts list
Connections:
- net +3.3V: now also SW2.2 (B); no longer C1.2, U3.3 (VI), U4.5 (BAT), U5.1 (EN), U5.10 (VIN), U5.2 (SEL)
- net 3.3V: now also R15.1, SW1.2
- net 5V: no longer U4.4 (V_{CC})
- net GND: now also J1.A1 (GND), J1.A12 (GND), J1.B1 (GND), J1.B12 (GND), J1.SH (SHIELD), Q3.1 (E), R12.2, R13.2
- net RST: now reaches U1.7 (~{RST})
- net RST: now also Q3.3 (C), R15.2
- new net: Q3.2 (B), SW1.1
- new net: J1.A5 (CC1), R13.1
- new net: J1.B5 (CC2), R12.1
- new net 3.3VRAW: C1.2, SW2.1 (A), U3.3 (VI), U4.5 (BAT), U5.1 (EN), U5.10 (VIN), U5.2 (SEL)
- new net UDM: J1.A7 (D-), J1.B7 (D-)
- new net UDP: J1.A6 (D+), J1.B6 (D+)
- new net USB5V: J1.A4 (VBUS), J1.A9 (VBUS), J1.B4 (VBUS), J1.B9 (VBUS), U4.4 (V_{CC})

Commit message: Updated journal to reflect wasted time on 3.3-5V converter, started work on additional memory schematic
Parts:
- added C3: C, symbol Device:C
- added R14: 10k, Resistor_SMD:R_0603_1608Metric, symbol Device:R
Connections:
- net 3.3V: now also R14.1
- net CS: now reaches U2.1 (~{CS})
- net CS: now also U1.14 (PA4)
- net at U2.3 (~{WP}/IO2): now also R14.2
Changed lines of the file:
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@@
+		)
+	)
+	(label "3.3V"
+		(at 115.57 130.81 180)
+		(effects
+			(font
+				(size 1.27 1.27)
+			)
+			(justify right bottom)
 		)
 	)
@@
 		)
 	)
+	(label "CS"
+		(at 64.77 43.18 0)
+		(effects
+			(font
+				(size 1.27 1.27)
+			)
+			(justify left bottom)
+		)
+	)
 	(label "3.3V"
 		(at 49.53 27.94 90)
@@
 			)
 			(justify left bottom)
+		)
+	)
+	(label "CS"
+		(at 123.19 120.65 180)
+		(effects
+			(font
+				(size 1.27 1.27)
+			)
+			(justify right bottom)
 		)
 	)
@@
 	)
 	(symbol
+		(lib_id "Device:C")
+		(at 162.56 128.27 0)
+		(unit 1)
+		(body_style 1)
+		(exclude_from_sim no)
+		(in_bom yes)
+		(on_board yes)
+		(in_pos_files yes)
+		(dnp no)
+		(fields_autoplaced yes)
+		(property "Reference" "C3"
+			(at 166.37 126.9999 0)
+			(show_name no)
+			(do_not_autoplace no)
+			(effects
+				(font
+					(size 1.27 1.27)
+				)
+				(justify left)
+			)
+		)
+		(property "Value" "C"
+			(at 166.37 129.5399 0)
+			(show_name no)
+			(do_not_autoplace no)
+			(effects
+				(font
+					(size 1.27 1.27)
+				)
+				(justify left)
+			)
+		)
+		(property "Footprint" ""
+			(at 163.5252 132.08 0)
+			(hide yes)
+			(show_name no)
+			(do_not_autoplace no)
+			(effects
+				(font
+					(size 1.27 1.27)
+				)
+			)
+		)
+		(property "Datasheet" ""
+			(at 162.56 128.27 0)
+			(hide yes)
+			(show_name no)
+			(do_not_autoplace no)
+			(effects
+				(font
+					(size 1.27 1.27)
+				)
+			)
+		)
+		(property "Description" "Unpolarized capacitor"
+			(at 162.56 128.27 0)
+			(hide yes)
+			(show_name no)
+			(do_not_autoplace no)
+			(effects
+				(font
+					(size 1.27 1.27)
+				)
+			)
+		)
+		(pin "2"
+		)
+		(pin "1"
+		)
+		(instances
+			(project "HyperPlex"
+				(path "/2159c24b-fff8-4711-9dc0-b98f0132545c"
+					(reference "C3")
+					(unit 1)
+				)
+			)
+		)
+	)
+	(symbol
 		(lib_id "Device:R")
 		(at 275.59 41.91 90)
@@
 					(unit 1)
 				)
+			)
+		)
+	)
+	(symbol
+		(lib_id "Device:R")
+		(at 119.38 130.81 90)
+		(unit 1)
+		(body_style 1)
+		(exclude_from_sim no)
+		(in_bom yes)
+		(on_board yes)
+		(in_pos_files yes)
+		(dnp no)
+		(property "Reference" "R14"
+			(at 119.38 132.842 90)
+			(show_name no)
+			(do_not_autoplace no)
+			(effects
+				(font
+					(size 1.27 1.27)
+				)
+			)
+		)
+		(property "Value" "10k"
+			(at 119.38 130.81 90)
+			(show_name no)
+			(do_not_autoplace no)
+			(effects
+				(font
+					(size 1.27 1.27)
+				)
+			)
+		)
+		(property "Footprint" "Resistor_SMD:R_0603_1608Metric"
+			(at 119.38 132.588 90)
+			(hide yes)
+			(show_name no)
+			(do_not_autoplace no)
+			(effects
+				(font
+					(size 1.27 1.27)
+				)
+			)
+		)
+		(property "Datasheet" ""
+			(at 119.38 130.81 0)
+			(hide yes)
+			(show_name no)
+			(do_not_autoplace no)
+			(effects
+				(font
+					(size 1.27 1.27)
+				)
+			)
+		)
+		(property "Description" "Resistor"
+			(at 119.38 130.81 0)
+			(hide yes)
+			(show_name no)
+			(do_not_autoplace no)
+			(effects
+				(font
+					(size 1.27 1.27)
+				)
+			)
+		)
+		(pin "1"
+		)
+		(pin "2"
+		)
+		(instances
+			(project "HyperPlex"
+				(path "/2159c24b-fff8-4711-9dc0-b98f0132545c"
+					(reference "R14")
+					(unit 1)
+				)

Commit message: Added journal entry 2, finished schematic, began PCB layout
Parts:
- removed C3: C, symbol Device:C
- removed U2: GD25QxxxEY, Package_SO:SOIC-8_5.3x5.3mm_P1.27mm, symbol Memory_Flash:GD25QxxxEY
- added SW3: SW_SPDT, Button_Switch_SMD:SW_SPDT_CK_JS102011SAQN, symbol Switch:SW_SPDT
- added SW4: SW_Push, Button_Switch_SMD:SW_SPST_PTS647_Sx38, symbol Switch:SW_Push
- added U6: XC6206PxxxMR, Package_TO_SOT_SMD:SOT-23, symbol Regulator_Linear:XC6206PxxxMR
- J1: footprint (none) -> Connector_USB:USB_C_Receptacle_G-Switch_GT-USB-7010ASV
- SW1: footprint (none) -> Button_Switch_SMD:SW_SPST_PTS647_Sx38
- SW2: footprint (none) -> Button_Switch_SMD:SW_SPDT_CK_JS102011SAQN
Connections:
- net UDM is gone; now on net USBDN: J1.A7 (D-), J1.B7 (D-)
- net UDP is gone; now on net USBDP: J1.A6 (D+), J1.B6 (D+)
- net 3.3V: now also SW3.2 (B), SW4.1; no longer R14.1, U3.2 (VO)
- net 5V: no longer U4.8 (CE)
- net GND: now also R14.1, U6.1 (GND)
- net USB5V: now also U4.8 (CE), U6.3 (VI)
- net at R14.2: now also U1.44 (BOOT0), SW4.2
- net USBDN: now reaches U1.32 (PA11)
- net USBDP: now reaches U1.33 (PA12)
- net CS: no longer names the net of U1.14 (PA4)
- new net: SW3.1 (A), U3.2 (VO)
- new net: SW3.3 (C), U6.2 (VO)
Other:
- moved on the sheet: U3

Commit message: Elaborated on journal, tentatively finished devboard PCB
Parts:
- R2: value 2.4k -> 1.5k
Changed lines of the file:
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@@
 			)
 		)
-		(property "Value" "2.4k"
+		(property "Value" "1.5k"
 			(at 275.59 44.45 90)
 			(show_name no)
